File: hardware/v1/simpleBJTtia.kicad_sch (KiCad schematic)
At the start: 28 parts, among them J101 +10V, J102 gnd, J103 Conn_Coaxial, J104 Conn_Coaxial, Q101 MMBFJ112, Q102 BC847

Commit message: Update project to kicad V9
Changed lines of the file:
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@@
 (kicad_sch
-	(version 20231120)
+	(version 20250114)
 	(generator "eeschema")
-	(generator_version "8.0")
+	(generator_version "9.0")
 	(paper "A4")
 	(junction
@@
 		)
 	)
+	(embedded_fonts no)
 )
