File: hardware/v2/v2.kicad_pcb (KiCad board)
At the start: 2 copper layers, 100 x 50 mm, 24 parts, among them J1 +10V, J2 gnd, J3 Conn_Coaxial, J4 Conn_Coaxial, Q1 MMBFJ112, Q2 MMBFJ112, Q3 BC847

Commit message: update v2
Parts:
- removed C2: 4u7, Capacitor_THT:C_Rect_L7.2mm_W5.5mm_P5.00mm_FKS2_FKP2_MKS2_MKP2
- C1, C4: value 4u7 -> 1u
- C3: value 33n -> 10n
Routing:
- net Net-(J4-In): track 35.2 -> 34.3 mm
