File: hardware/v2/v2.kicad_sch (KiCad schematic)
At the start: 24 parts, among them J1 +10V, J2 gnd, J3 Conn_Coaxial, J4 Conn_Coaxial, Q1 MMBFJ112, Q2 MMBFJ112, Q3 BC847

Commit message: update v2
Parts:
- removed C2: 4u7, Capacitor_THT:C_Rect_L7.2mm_W5.5mm_P5.00mm_FKS2_FKP2_MKS2_MKP2, symbol Device:C
- C1, C4: value 4u7 -> 1u
- C3: value 33n -> 10n
Changed lines of the file:
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@@
-	)
-	(junction
-		(at 81.28 38.1)
-		(diameter 0)
-		(color 0 0 0 0)
 	)
 	(junction
@@
 	(wire
 		(pts
-			(xy 81.28 38.1) (xy 121.92 38.1)
-		)
-		(stroke
-			(width 0)
-			(type default)
-		)
-	)
-	(wire
-		(pts
 			(xy 137.16 72.39) (xy 137.16 52.07)
 		)
@@
 	(wire
 		(pts
-			(xy 81.28 40.64) (xy 81.28 38.1)
-		)
-		(stroke
-			(width 0)
-			(type default)
-		)
-	)
-	(wire
-		(pts
 			(xy 168.91 113.03) (xy 168.91 109.22)
 		)
@@
 	(wire
 		(pts
-			(xy 81.28 50.8) (xy 81.28 48.26)
-		)
-		(stroke
-			(width 0)
-			(type default)
-		)
-	)
-	(wire
-		(pts
 			(xy 121.92 74.93) (xy 121.92 72.39)
 		)
@@
 	(wire
 		(pts
-			(xy 67.31 38.1) (xy 81.28 38.1)
+			(xy 67.31 38.1) (xy 121.92 38.1)
 		)
 		(stroke
@@
 			)
 		)
-		(property "Value" "4u7"
+		(property "Value" "1u"
 			(at 151.13 107.95 90)
 			(effects
@@
 				(path "/e52b76a6-63dd-465f-8d19-818dbe6e1d51"
 					(reference "C6")
-					(unit 1)
-				)
-			)
-		)
-	)
-	(symbol
-		(lib_id "Device:C")
-		(at 81.28 44.45 180)
-		(unit 1)
-		(exclude_from_sim no)
-		(in_bom yes)
-		(on_board yes)
-		(dnp no)
-		(fields_autoplaced yes)
-		(property "Reference" "C2"
-			(at 85.09 43.1799 0)
-			(effects
-				(font
-					(size 1.27 1.27)
-				)
-				(justify right)
-			)
-		)
-		(property "Value" "4u7"
-			(at 85.09 45.7199 0)
-			(effects
-				(font
-					(size 1.27 1.27)
-				)
-				(justify right)
-			)
-		)
-		(property "Footprint" "Capacitor_THT:C_Rect_L7.2mm_W5.5mm_P5.00mm_FKS2_FKP2_MKS2_MKP2"
-			(at 80.3148 40.64 0)
-			(effects
-				(font
-					(size 1.27 1.27)
-				)
-				(hide yes)
-			)
-		)
-		(property "Datasheet" "~"
-			(at 81.28 44.45 0)
-			(effects
-				(font
-					(size 1.27 1.27)
-				)
-				(hide yes)
-			)
-		)
-		(property "Description" "Unpolarized capacitor"
-			(at 81.28 44.45 0)
-			(effects
-				(font
-					(size 1.27 1.27)
-				)
-				(hide yes)
-			)
-		)
-		(pin "1"
-		)
-		(pin "2"
-		)
-		(instances
-			(project "v2"
-				(path "/e52b76a6-63dd-465f-8d19-818dbe6e1d51"
-					(reference "C2")
 					(unit 1)
 				)
@@
 				(path "/e52b76a6-63dd-465f-8d19-818dbe6e1d51"
 					(reference "Q3")
-					(unit 1)
-				)
-			)
-		)
-	)
-	(symbol
-		(lib_id "power:GND")
-		(at 81.28 50.8 0)
-		(unit 1)
-		(exclude_from_sim no)
-		(in_bom yes)
-		(on_board yes)
-		(dnp no)
-		(fields_autoplaced yes)
-		(property "Reference" "#PWR05"
-			(at 81.28 57.15 0)
-			(effects
-				(font
-					(size 1.27 1.27)
-				)
-				(hide yes)
-			)
-		)
-		(property "Value" "GND"
-			(at 81.28 55.88 0)
-			(effects
-				(font
-					(size 1.27 1.27)
-				)
-			)
-		)
-		(property "Footprint" ""
-			(at 81.28 50.8 0)
-			(effects
-				(font
-					(size 1.27 1.27)
-				)
-				(hide yes)
-			)
-		)
-		(property "Datasheet" ""
-			(at 81.28 50.8 0)
-			(effects
-				(font
-					(size 1.27 1.27)
-				)
-				(hide yes)
-			)
-		)
-		(property "Description" "Power symbol creates a global label with name \"GND\" , ground"
-			(at 81.28 50.8 0)
-			(effects
-				(font
-					(size 1.27 1.27)
-				)
-				(hide yes)
-			)
-		)
-		(pin "1"
-		)
-		(instances
-			(project "v2"
-				(path "/e52b76a6-63dd-465f-8d19-818dbe6e1d51"
-					(reference "#PWR05")
 					(unit 1)
 				)
@@
 			)
 		)
-		(property "Value" "33n"
+		(property "Value" "10n"
 			(at 102.87 102.8699 0)
 			(effects
@@
 			)
 		)
-		(property "Value" "4u7"
+		(property "Value" "1u"
 			(at 71.12 45.7199 0)
 			(effects
