File: hardware/howNotTo/howNotTo.kicad_sch (KiCad schematic)
At the start: 22 parts, among them J1 +10V, J2 gnd, J3 Conn_Coaxial, J4 Conn_Coaxial, Q3 BC847

Commit message: update the how not to design
Parts:
- removed C2: 4u7, Capacitor_THT:C_Rect_L7.2mm_W5.5mm_P5.00mm_FKS2_FKP2_MKS2_MKP2, symbol Device:C
- C1, C3, C5, C6, C7: value 4u7 -> 1u
- R3: value 11k5 -> 12k
Changed lines of the file:
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@@
 		(color 0 0 0 0)
 	)
-	(junction
-		(at 101.6 38.1)
-		(diameter 0)
-		(color 0 0 0 0)
-	)
 	(wire
 		(pts
@@
 	(wire
 		(pts
-			(xy 88.9 38.1) (xy 101.6 38.1)
+			(xy 88.9 38.1) (xy 114.3 38.1)
 		)
 		(stroke
@@
 	(wire
 		(pts
-			(xy 101.6 53.34) (xy 101.6 49.53)
-		)
-		(stroke
-			(width 0)
-			(type default)
-		)
-	)
-	(wire
-		(pts
 			(xy 165.1 101.6) (xy 165.1 105.41)
 		)
@@
 	(wire
 		(pts
-			(xy 101.6 38.1) (xy 114.3 38.1)
-		)
-		(stroke
-			(width 0)
-			(type default)
-		)
-	)
-	(wire
-		(pts
 			(xy 191.77 76.2) (xy 191.77 83.82)
 		)
@@
 		(pts
 			(xy 124.46 104.14) (xy 124.46 95.25)
-		)
-		(stroke
-			(width 0)
-			(type default)
-		)
-	)
-	(wire
-		(pts
-			(xy 101.6 41.91) (xy 101.6 38.1)
 		)
 		(stroke
@@
 	(symbol
 		(lib_id "Device:C")
-		(at 101.6 45.72 180)
-		(unit 1)
-		(exclude_from_sim no)
-		(in_bom yes)
-		(on_board yes)
-		(dnp no)
-		(fields_autoplaced yes)
-		(property "Reference" "C2"
-			(at 105.41 44.4499 0)
-			(effects
-				(font
-					(size 1.27 1.27)
-				)
-				(justify right)
-			)
-		)
-		(property "Value" "4u7"
-			(at 105.41 46.9899 0)
-			(effects
-				(font
-					(size 1.27 1.27)
-				)
-				(justify right)
-			)
-		)
-		(property "Footprint" "Capacitor_THT:C_Rect_L7.2mm_W5.5mm_P5.00mm_FKS2_FKP2_MKS2_MKP2"
-			(at 100.6348 41.91 0)
-			(effects
-				(font
-					(size 1.27 1.27)
-				)
-				(hide yes)
-			)
-		)
-		(property "Datasheet" "~"
-			(at 101.6 45.72 0)
-			(effects
-				(font
-					(size 1.27 1.27)
-				)
-				(hide yes)
-			)
-		)
-		(property "Description" "Unpolarized capacitor"
-			(at 101.6 45.72 0)
-			(effects
-				(font
-					(size 1.27 1.27)
-				)
-				(hide yes)
-			)
-		)
-		(pin "2"
-		)
-		(pin "1"
-		)
-		(instances
-			(project ""
-				(path "/bd9d1afa-a1ef-4266-8ae3-21cf7d8b6d9f"
-					(reference "C2")
-					(unit 1)
-				)
-			)
-		)
-	)
-	(symbol
-		(lib_id "Device:C")
 		(at 133.35 133.35 90)
 		(unit 1)
@@
 	)
 	(symbol
-		(lib_id "power:GND")
-		(at 101.6 53.34 0)
-		(unit 1)
-		(exclude_from_sim no)
-		(in_bom yes)
-		(on_board yes)
-		(dnp no)
-		(fields_autoplaced yes)
-		(property "Reference" "#PWR04"
-			(at 101.6 59.69 0)
-			(effects
-				(font
-					(size 1.27 1.27)
-				)
-				(hide yes)
-			)
-		)
-		(property "Value" "GND"
-			(at 101.6 58.42 0)
-			(effects
-				(font
-					(size 1.27 1.27)
-				)
-			)
-		)
-		(property "Footprint" ""
-			(at 101.6 53.34 0)
-			(effects
-				(font
-					(size 1.27 1.27)
-				)
-				(hide yes)
-			)
-		)
-		(property "Datasheet" ""
-			(at 101.6 53.34 0)
-			(effects
-				(font
-					(size 1.27 1.27)
-				)
-				(hide yes)
-			)
-		)
-		(property "Description" "Power symbol creates a global label with name \"GND\" , ground"
-			(at 101.6 53.34 0)
-			(effects
-				(font
-					(size 1.27 1.27)
-				)
-				(hide yes)
-			)
-		)
-		(pin "1"
-		)
-		(instances
-			(project "howNotTo"
-				(path "/bd9d1afa-a1ef-4266-8ae3-21cf7d8b6d9f"
-					(reference "#PWR04")
-					(unit 1)
-				)
-			)
-		)
-	)
-	(symbol
 		(lib_id "Device:C")
 		(at 157.48 63.5 90)
@@
 			)
 		)
-		(property "Value" "4u7"
+		(property "Value" "1u"
 			(at 157.48 58.42 90)
 			(effects
@@
 			)
 		)
-		(property "Value" "4u7"
+		(property "Value" "1u"
 			(at 92.71 46.9899 0)
 			(effects
@@
 			)
 		)
-		(property "Value" "4u7"
+		(property "Value" "1u"
 			(at 156.21 99.0599 0)
 			(effects
@@
 			)
 		)
-		(property "Value" "4u7"
+		(property "Value" "1u"
 			(at 168.91 99.0599 0)
 			(effects
@@
 			)
 		)
-		(property "Value" "11k5"
+		(property "Value" "12k"
 			(at 127 92.7099 0)
 			(effects
@@
 			)
 		)
-		(property "Value" "4u7"
+		(property "Value" "1u"
 			(at 102.87 71.12 90)
 			(effects
