File: hardware/V4/V4.kicad_pcb (KiCad board)
At the start: 4 copper layers, 250 x 100 mm, 122 parts, among them J1 Uraw, J10 Enable channel, J11 Enable channel, J12 Output, J13 Output, J14 Output, J15 Output, J16 Select psu filter, J17 IndCoupling, J18 CapCoupling, J19 GND, J2 Inductive coupling, J3 Capacitive coupling, J4 Input, J5 Input, J6 Input, J7 Input, J8 Enable channel, J9 Enable channel, Q1 DMP2123L-7, Q10 MMBFJ112, Q11 MMBFJ112, Q12 MMBFJ112, Q13 BCM856BSH-Q, Q14 MMBFJ112, Q15 MMBFJ112, Q16 MMBFJ112, Q17 2PD601ARL, Q18 MMBFJ112, Q19 2PD601ARL, Q2 MMBFJ112, Q20 2PD601ARL, Q3 MMBFJ112, Q4 MMBFJ112, Q5 BCM856BSH-Q, Q6 MMBFJ112, Q7 MMBFJ112, Q8 MMBFJ112, Q9 2PD601ARL

Commit message: Adding initial v4 design
Parts:
- J17, J18: footprint Connector_PinSocket_2.54mm:PinSocket_1x02_P2.54mm_Vertical -> Connector_PinHeader_2.54mm:PinHeader_1x02_P2.54mm_Vertical
- L1: value L -> 10m
- L2: value L -> 10u
- moved D8 50.8 mm to (109.5, 59.8)
- moved J12 40.0 mm to (110.0, 55.0)
- moved J13 40.0 mm to (150.0, 55.5)
- moved D9 38.8 mm to (149.5, 60.2)
- moved C20 28.2 mm to (183.5, 98.5)
- moved R24 27.6 mm to (189.1, 115.2), turned to 180 degrees
- moved C19 27.5 mm to (189.1, 117.5), turned to 180 degrees
- moved J3 26.2 mm to (75.0, 125.0)
- moved D3 26.1 mm to (76.0, 120.0)
- moved C18 26.1 mm to (190.0, 112.0)
- moved C21 26.1 mm to (193.5, 96.5)
- moved Q19 26.1 mm to (189.0, 99.5)
- moved R21 26.1 mm to (191.0, 104.0)
- moved R23 26.1 mm to (191.0, 106.5)
- moved R26 26.1 mm to (193.5, 99.0)
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Routing:
- net /4 resistor biased transimpedance amplifier 2/out: track 0.00 -> 75.9 mm
- net /4 resistor biased transimpedance amplifier 1/out: track 0.00 -> 75.9 mm
- net /Current biased transimpedance amplifier 1/out: track 0.00 -> 68.6 mm
- net /Current biased transimpedance amplifier 2/out: track 0.00 -> 68.5 mm
- net GND: track 0.00 -> 55.9 mm, vias 0 -> 224
- net Net-(C1-+): track 0.00 -> 35.7 mm
- net Net-(J16-Pin_5): track 0.00 -> 31.8 mm
- net /power/CapacitiveCoupling: track 0.00 -> 28.0 mm
- net Net-(C2-+): track 0.00 -> 27.3 mm
- net Net-(J17-Pin_2): track 0.00 -> 19.0 mm
- net /Current biased transimpedance amplifier 2/in: track 0.00 -> 12.9 mm
- net Net-(C17-+): track 0.00 -> 12.5 mm
- net Net-(C11-+): track 0.00 -> 12.5 mm
- net /Current biased transimpedance amplifier 1/in: track 0.00 -> 12.4 mm
- net /4 resistor biased transimpedance amplifier 1/in: track 0.00 -> 12.1 mm
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- added copper zone on F.Cu, net /4 resistor biased transimpedance amplifier 1/Usup
- added copper zone on F.Cu, net /4 resistor biased transimpedance amplifier 2/Usup
- added copper zone on F.Cu, net /Current biased transimpedance amplifier 1/Usup
- added copper zone on F.Cu, net /Current biased transimpedance amplifier 2/Usup
- added copper zone on F.Cu, net /power/Uraw
- added copper zone on B.Cu, net /power/Usup
- added copper zone on B.Cu, net GND
- added copper zone on F.Cu, net GND
- added copper zone on In1.Cu, net GND
- added copper zone on In2.Cu, net GND
- added copper zone on F.Cu, net Net-(D12-K)
Other:
- board size 250 x 100 mm -> 240 x 100 mm
- board text added: "1"
- board text added: "2"
- board text added: "3"
- board text added: "4"
- board text added: "4 resistor biasing"
- board text added: "5"
- board text added: "Biasing effect on EMC"
- board text added: "Capacitive coupling"
- board text added: "Chan 1"
- board text added: "Chan 2"
- board text added: "Chan 3"
- board text added: "Chan 4"
- board text added: "Current biasing"
- board text added: "Enable channel"
- board text added: "ID"
- board text added: "Inductive coupling"
- board text added: "Rev 1"
- board text added: "TychoJ"
- board text added: "https://tychoj.com"
