File: hardware/V4/power.kicad_sch (KiCad schematic)
At the start: 19 parts, among them J16 Select psu filter, J17 IndCoupling, J18 CapCoupling, Q1 DMP2123L-7, Q2 MMBFJ112

Commit message: Adding initial v4 design
Parts:
- J17, J18: footprint Connector_PinSocket_2.54mm:PinSocket_1x02_P2.54mm_Vertical -> Connector_PinHeader_2.54mm:PinHeader_1x02_P2.54mm_Vertical
- L1: value L -> 10m
- L2: value L -> 10u
Other:
- note added: "Select power supply filters"
- moved on the sheet: R1
Changed lines of the file:
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@@
 	(paper "A4")
+	(rectangle
+		(start 100.33 25.4)
+		(end 181.61 129.54)
+		(stroke
+			(width 0)
+			(type dash)
+		)
+		(fill
+			(type none)
+		)
+	)
 	(rectangle
 		(start 36.83 85.09)
@@
 		)
 	)
+	(text "Select power supply filters"
+		(exclude_from_sim no)
+		(at 136.906 27.686 0)
+		(effects
+			(font
+				(size 1.27 1.27)
+			)
+		)
+	)
 	(junction
 		(at 124.46 71.12)
@@
 	(wire
 		(pts
-			(xy 66.04 147.32) (xy 66.04 153.67)
+			(xy 66.04 147.32) (xy 66.04 151.13)
 		)
 		(stroke
@@
 	(wire
 		(pts
-			(xy 66.04 163.83) (xy 66.04 165.1)
+			(xy 66.04 161.29) (xy 66.04 165.1)
 		)
 		(stroke
@@
 			)
 		)
-		(property "Footprint" "Connector_PinSocket_2.54mm:PinSocket_1x02_P2.54mm_Vertical"
+		(property "Footprint" "Connector_PinHeader_2.54mm:PinHeader_1x02_P2.54mm_Vertical"
 			(at 215.9 109.22 0)
 			(effects
@@
 	(symbol
 		(lib_id "PCM_Elektuur:R")
-		(at 66.04 158.75 0)
+		(at 66.04 156.21 0)
 		(unit 1)
 		(exclude_from_sim no)
@@
 		(fields_autoplaced yes)
 		(property "Reference" "R1"
+			(at 68.58 154.9399 0)
+			(effects
+				(font
+					(size 1.27 1.27)
+				)
+				(justify left)
+			)
+		)
+		(property "Value" "1k"
 			(at 68.58 157.4799 0)
 			(effects
@@
 			)
 		)
-		(property "Value" "1k"
-			(at 68.58 160.0199 0)
-			(effects
-				(font
-					(size 1.27 1.27)
-				)
-				(justify left)
-			)
-		)
 		(property "Footprint" "Resistor_SMD:R_0805_2012Metric"
-			(at 66.04 158.75 0)
+			(at 66.04 156.21 0)
 			(effects
 				(font
@@
 		)
 		(property "Datasheet" ""
-			(at 66.04 158.75 0)
+			(at 66.04 156.21 0)
 			(effects
 				(font
@@
 		)
 		(property "Description" "resistor"
-			(at 66.04 158.75 0)
+			(at 66.04 156.21 0)
 			(effects
 				(font
@@
 		)
 		(property "Indicator" "+"
-			(at 62.865 155.575 0)
+			(at 62.865 153.035 0)
 			(effects
 				(font
@@
 		)
 		(property "Rating" "W"
-			(at 68.58 161.925 0)
+			(at 68.58 159.385 0)
 			(effects
 				(font
@@
 			)
 		)
-		(property "Value" "L"
+		(property "Value" "10u"
 			(at 116.84 67.31 90)
 			(effects
@@
 			)
 		)
-		(property "Value" "L"
+		(property "Value" "10m"
 			(at 116.84 52.07 90)
 			(effects
@@
 			)
 		)
-		(property "Footprint" "Connector_PinSocket_2.54mm:PinSocket_1x02_P2.54mm_Vertical"
+		(property "Footprint" "Connector_PinHeader_2.54mm:PinHeader_1x02_P2.54mm_Vertical"
 			(at 199.39 109.22 0)
 			(effects
